Commit message: Update visual for MPU6050 with rotated origin

File: urdf/mpu6050.urdf.xacro (robot description, xacro)
@@ -4,16 +4,18 @@
   <link name="imu">
     <visual>
-      <origin xyz="0.05 0 0" rpy="0 0 -1.5708" />
+      <origin xyz="0.0 0 0" rpy="0 0 0" />
       <geometry>
-        <box size="0.5 0.5 0.25"/>
+        <box size="1 0.8 0.5"/>
       </geometry>
       <material name="black">
-        <color rgba="0 0 0  1"/>
+        <color rgba="0.5 0.5 0.5  0.5"/>
       </material>
     </visual>
+  </link>
+  <link name="imu_model">
     <visual>
-      <origin xyz="0 0 0" rpy="0 0 -1.5708" />
+      <origin xyz="0 0 0" rpy="0 0 0" />
       <geometry>
-        <mesh filename="package://mpu6050_ros/meshes/mpu6050/mpu6050.stl" scale="0.1 0.1 0.1"/>
+        <mesh filename="package://mpu6050_ros/meshes/mpu6050/mpu6050.stl" scale="0.01 0.01 0.01"/>
       </geometry>
       <material name="darkblue">
@@ -22,4 +24,9 @@
     </visual>
   </link>
+  <joint name="imu_to_imu_model" type="fixed">
+    <origin xyz="0 0 0" rpy="0 0 0" />
+    <parent link="imu" />
+    <child link="imu_model" />
+  </joint>
   <joint name="world_to_imu" type="fixed">
     <origin xyz="0 0 0" rpy="0 0 0" />
